Commit message: add dynamixel training & stl conv

File: dynamics/src/dynamics/urdf/random.urdf (robot description, URDF)
Before this commit: robot tecobot, 8 links, 7 joints
Links:
- link 2: mass 1.6876153475434592 -> 1.6508092151221665
- link 3: mass 0.5460670914510587 -> 0.4964628887269289
Joints:
- joint j3: origin xyz=0 0.24825321185198293 0 rpy=0 0 0 -> xyz=0 0.14038412276640627 0 rpy=0 0 0
- joint j4: origin xyz=0 0.454138963226822 0.0203999999999699 rpy=1.57079632675385 0 -3.14159265356591 -> xyz=0 0.3087620977245759 0.0203999999999699 rpy=1.57079632675385 0 -3.14159265356591

File: dynamics/src/dynamics/urdf/single_arm_v12.urdf (robot description, URDF)
Before this commit: robot single_arm_v12, 8 links, 7 joints
Links:
- link Link2: mass 0.61539 -> 0.44844344500975386; geometry collision mesh filename=package://single_arm_v12/meshes/Link2.STL; visual mesh filename=package://dynamics/src/dynamics/meshes/single_arm_v12_2_12.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
- link Link3: mass 0.558726771182515 -> 0.41466376837106494; geometry collision mesh filename=package://single_arm_v12/meshes/Link3.STL; visual mesh filename=package://dynamics/src/dynamics/meshes/single_arm_v12_3_12.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
Joints:
- joint Joint3: origin xyz=0.214 0 -0.0325 rpy=0 0 0 -> xyz=0.25214453759208827 0 -0.0325 rpy=0 0 0
- joint Joint4: origin xyz=0.214 0 0.0325 rpy=0 0 3.1416 -> xyz=0.27476925248418915 0 0.0325 rpy=0 0 3.1416
