Commit message: test motion planning

File: dynamics/src/dynamics/urdf/single_arm_v12_motion.urdf (robot description, URDF)
Before this commit: robot single_arm_v12, 8 links, 7 joints
Links:
- link Link2: geometry collision mesh filename=package://dynamics/src/dynamics/meshes/merged_single_arm_ax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; visual mesh filename=package://dynamics/src/dynamics/meshes/merged_single_arm_ax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
- link Link3: geometry collision mesh filename=package://dynamics/src/dynamics/meshes/merged_single_arm_ax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; visual mesh filename=package://dynamics/src/dynamics/meshes/merged_single_arm_ax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

Commit message: fixed motion planning test

File: dynamics/src/dynamics/urdf/single_arm_v12_motion.urdf (robot description, URDF)
Before this commit: robot single_arm_v12, 8 links, 7 joints
Joints:
- joint Joint6: origin xyz=0.0346 0.068329 -0.0048371 rpy=1.5708 -1.5708 0 -> xyz=0.0346 0.0685 0 rpy=1.5708 -1.5708 0
