Commit message: add case 2 3,5dof actio & reset

File: dynamics/src/dynamics/urdf/single_arm_v12_motion_3dof.urdf (robot description, URDF)
Before this commit: robot single_arm_v12, 8 links, 7 joints
Links:
- removed link Link4
- removed link Link5
- removed link Link6
- link Link2: geometry collision mesh filename=package://dynamics/src/dynamics/meshes/merged_single_arm_ax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; visual mesh filename=package://dynamics/src/dynamics/meshes/merged_single_arm_ax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
- link Link3: geometry collision mesh filename=package://dynamics/src/dynamics/meshes/merged_single_arm_ax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; visual mesh filename=package://dynamics/src/dynamics/meshes/merged_single_arm_ax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
Joints:
- removed joint Joint4
- removed joint Joint5
- removed joint Joint6
