Commit message: fixed dynamixel robot DH& urdf include

File: dynamics/src/dynamics/urdf/single_arm_v12.urdf (robot description, URDF)
Before this commit: robot single_arm_v11, 8 links, 7 joints
Links:
- link Link1: geometry collision mesh filename=package://single_arm_v12/meshes/Link1.STL; visual mesh filename=package://single_arm_v12/meshes/Link1.STL
- link Link2: geometry collision mesh filename=package://single_arm_v12/meshes/Link2.STL; visual mesh filename=package://single_arm_v12/meshes/Link2.STL
- link Link3: mass 0.55872677113484 -> 0.558726771182515; geometry collision mesh filename=package://single_arm_v12/meshes/Link3.STL; visual mesh filename=package://single_arm_v12/meshes/Link3.STL
- link Link4: mass 0.31385 -> 0.313854171959486; geometry collision mesh filename=package://single_arm_v12/meshes/Link4.STL; visual mesh filename=package://single_arm_v12/meshes/Link4.STL
- link Link5: geometry collision mesh filename=package://single_arm_v12/meshes/Link5.STL; visual mesh filename=package://single_arm_v12/meshes/Link5.STL
- link Link6: mass 5.55809350532545 -> 5.5581; geometry collision mesh filename=package://single_arm_v12/meshes/Link6.STL; visual mesh filename=package://single_arm_v12/meshes/Link6.STL
- link base_link: geometry collision mesh filename=package://single_arm_v12/meshes/base_link.STL; visual mesh filename=package://single_arm_v12/meshes/base_link.STL
Joints:
- joint Joint1: origin xyz=-0.006708 -0.126 0.067093 rpy=0 0 -1.5001 -> xyz=0 0 0.1445 rpy=0 0 0
- joint Joint4: origin xyz=0.214 0 0.0325 rpy=0 0 0 -> xyz=0.214 0 0.0325 rpy=0 0 3.1416
- joint Joint5: axis 0 0 -1 -> -1 0 0; origin xyz=0 -0.0685 0.0346 rpy=1.5708 0 0 -> xyz=0 0.0685 0.0346 rpy=1.5708 0 1.5708
- joint Joint6: origin xyz=0 0.0685 0.0346 rpy=-1.5708 0 0 -> xyz=0.0346 0.068329 -0.0048371 rpy=3.1416 1.5001 -1.5708

File: single_arm_v12/urdf/single_arm_v12.urdf (robot description, URDF)
Before this commit: robot single_arm_v11, 8 links, 7 joints
Links:
- removed link dummy
- link Link1: geometry collision mesh filename=package://single_arm_v12/meshes/Link1.STL; visual mesh filename=package://single_arm_v12/meshes/Link1.STL
- link Link2: geometry collision mesh filename=package://single_arm_v12/meshes/Link2.STL; visual mesh filename=package://single_arm_v12/meshes/Link2.STL
- link Link3: mass 0.55872677113484 -> 0.558726771182515; geometry collision mesh filename=package://single_arm_v12/meshes/Link3.STL; visual mesh filename=package://single_arm_v12/meshes/Link3.STL
- link Link4: mass 0.31385 -> 0.313854171959486; geometry collision mesh filename=package://single_arm_v12/meshes/Link4.STL; visual mesh filename=package://single_arm_v12/meshes/Link4.STL
- link Link5: geometry collision mesh filename=package://single_arm_v12/meshes/Link5.STL; visual mesh filename=package://single_arm_v12/meshes/Link5.STL
- link Link6: mass 5.55809350532545 -> 5.5581; geometry collision mesh filename=package://single_arm_v12/meshes/Link6.STL; visual mesh filename=package://single_arm_v12/meshes/Link6.STL
- link base_link: geometry collision mesh filename=package://single_arm_v12/meshes/base_link.STL; visual mesh filename=package://single_arm_v12/meshes/base_link.STL
Joints:
- removed joint dummy_joint
- joint Joint1: origin xyz=-0.006708 -0.126 0.067093 rpy=0 0 -1.5001 -> xyz=0 0 0.1445 rpy=0 0 0
- joint Joint4: origin xyz=0.214 0 0.0325 rpy=0 0 0 -> xyz=0.214 0 0.0325 rpy=0 0 3.1416
- joint Joint5: axis 0 0 -1 -> -1 0 0; origin xyz=0 -0.0685 0.0346 rpy=1.5708 0 0 -> xyz=0 0.0685 0.0346 rpy=1.5708 0 1.5708
- joint Joint6: origin xyz=0 0.0685 0.0346 rpy=-1.5708 0 0 -> xyz=0.0346 0.068329 -0.0048371 rpy=3.1416 1.5001 -1.5708

Commit message: fixed cost & weight input &action

File: dynamics/src/dynamics/urdf/single_arm_v12.urdf (robot description, URDF)
Before this commit: robot single_arm_v12, 8 links, 7 joints
Links:
- link Link2: mass 0.44844344500975386 -> 0.44094844957718515
- link Link3: mass 0.41466376837106494 -> 0.3817208533320915
Joints:
- joint Joint3: origin xyz=0.25214453759208827 0 -0.0325 rpy=0 0 0 -> xyz=0.22261611424885444 0 -0.0325 rpy=0 0 0
- joint Joint4: origin xyz=0.27476925248418915 0 0.0325 rpy=0 0 3.1416 -> xyz=0.14498234925487014 0 0.0325 rpy=0 0 3.1416

Commit message: 改用IK LMS & 修改reward

File: dynamics/src/dynamics/urdf/single_arm_v12.urdf (robot description, URDF)
Before this commit: robot single_arm_v12, 8 links, 7 joints
Links:
- link Link2: mass 0.44094844957718515 -> 0.42388797186464855
- link Link3: mass 0.3817208533320915 -> 0.4393496937084793
Joints:
- joint Joint3: origin xyz=0.22261611424885444 0 -0.0325 rpy=0 0 0 -> xyz=0.1554020628373607 0 -0.0325 rpy=0 0 0
- joint Joint4: origin xyz=0.14498234925487014 0 0.0325 rpy=0 0 3.1416 -> xyz=0.372025667076 0 0.0325 rpy=0 0 3.1416

Commit message: remote cost&weight & fixed reward

File: dynamics/src/dynamics/urdf/single_arm_v12.urdf (robot description, URDF)
Before this commit: robot single_arm_v12, 8 links, 7 joints
Links:
- link Link2: mass 0.42388797186464855 -> 0.4247115169460981
- link Link3: mass 0.4393496937084793 -> 0.42969116545891584
Joints:
- joint Joint3: origin xyz=0.1554020628373607 0 -0.0325 rpy=0 0 0 -> xyz=0.15864662622983572 0 -0.0325 rpy=0 0 0
- joint Joint4: origin xyz=0.372025667076 0 0.0325 rpy=0 0 3.1416 -> xyz=0.33397346465916106 0 0.0325 rpy=0 0 3.1416

Commit message: add 4,5,6 dof robot model

File: dynamics/src/dynamics/urdf/single_arm_v12.urdf (robot description, URDF)
Before this commit: robot single_arm_v12, 8 links, 7 joints
Links:
- link Link2: mass 0.4247115169460981 -> 0.4495799720620618
- link Link3: mass 0.42969116545891584 -> 0.41352459447819634
Joints:
- joint Joint3: origin xyz=0.15864662622983572 0 -0.0325 rpy=0 0 0 -> xyz=0.25662217233429996 0 -0.0325 rpy=0 0 0
- joint Joint4: origin xyz=0.33397346465916106 0 0.0325 rpy=0 0 3.1416 -> xyz=0.27028119028264486 0 0.0325 rpy=0 0 3.1416

Commit message: fixed reach_manipulability_evaluate  count = 0

File: dynamics/src/dynamics/urdf/single_arm_v12.urdf (robot description, URDF)
Before this commit: robot single_arm_v12, 8 links, 7 joints
Links:
- link Link2: mass 0.4495799720620618 -> 0.43774308917126725
- link Link3: mass 0.41352459447819634 -> 0.4023794007282979
Joints:
- joint Joint3: origin xyz=0.25662217233429996 0 -0.0325 rpy=0 0 0 -> xyz=0.20998778913710137 0 -0.0325 rpy=0 0 0
- joint Joint4: origin xyz=0.27028119028264486 0 0.0325 rpy=0 0 3.1416 -> xyz=0.22637189503725522 0 0.0325 rpy=0 0 3.1416

Commit message: design reward function version1

File: dynamics/src/dynamics/urdf/single_arm_v12.urdf (robot description, URDF)
Before this commit: robot single_arm_v12, 8 links, 7 joints
Links:
- link Link2: mass 0.43774308917126725 -> 0.44921843295062003
- link Link3: mass 0.4023794007282979 -> 0.444800458017923
Joints:
- joint Joint3: origin xyz=0.20998778913710137 0 -0.0325 rpy=0 0 0 -> xyz=0.2551977978922024 0 -0.0325 rpy=0 0 0
- joint Joint4: origin xyz=0.22637189503725522 0 0.0325 rpy=0 0 3.1416 -> xyz=0.3935003246501293 0 0.0325 rpy=0 0 3.1416

Commit message: add test model select input

File: dynamics/src/dynamics/urdf/single_arm_v12.urdf (robot description, URDF)
Before this commit: robot single_arm_v12, 8 links, 7 joints
Links:
- link Link2: mass 0.44921843295062003 -> 0.49844869339364356
- link Link3: mass 0.444800458017923 -> 0.40709071786215845
Joints:
- joint Joint3: origin xyz=0.2551977978922024 0 -0.0325 rpy=0 0 0 -> xyz=0.44915281557538766 0 -0.0325 rpy=0 0 0
- joint Joint4: origin xyz=0.3935003246501293 0 0.0325 rpy=0 0 3.1416 -> xyz=0.2449333143959118 0 0.0325 rpy=0 0 3.1416

Commit message: ddqn_train_eps & tested return current design

File: dynamics/src/dynamics/urdf/single_arm_v12.urdf (robot description, URDF)
Before this commit: robot single_arm_v12, 8 links, 7 joints
Links:
- link Link2: mass 0.49844869339364356 -> 0.4560060691069818
- link Link3: mass 0.40709071786215845 -> 0.4243988698152576
Joints:
- joint Joint3: origin xyz=0.44915281557538766 0 -0.0325 rpy=0 0 0 -> xyz=0.28193940110305304 0 -0.0325 rpy=0 0 0
- joint Joint4: origin xyz=0.2449333143959118 0 0.0325 rpy=0 0 3.1416 -> xyz=0.3131231342694003 0 0.0325 rpy=0 0 3.1416

Commit message: fixed reward

File: dynamics/src/dynamics/urdf/single_arm_v12.urdf (robot description, URDF)
Before this commit: robot single_arm_v12, 8 links, 7 joints
Links:
- link Link2: mass 0.4560060691069818 -> 0.4982976067496825
- link Link3: mass 0.4243988698152576 -> 0.44424181816446623
Joints:
- joint Joint3: origin xyz=0.28193940110305304 0 -0.0325 rpy=0 0 0 -> xyz=0.44855757166569743 0 -0.0325 rpy=0 0 0
- joint Joint4: origin xyz=0.3131231342694003 0 0.0325 rpy=0 0 3.1416 -> xyz=0.39129942237676174 0 0.0325 rpy=0 0 3.1416

Commit message: fixed axis length action space negative value

File: dynamics/src/dynamics/urdf/single_arm_v12.urdf (robot description, URDF)
Before this commit: robot single_arm_v12, 8 links, 7 joints
Links:
- link Link2: mass 0.4982976067496825 -> 0.5043461294231942
- link Link3: mass 0.44424181816446623 -> 0.4691908056563082
Joints:
- joint Joint3: origin xyz=0.44855757166569743 0 -0.0325 rpy=0 0 0 -> xyz=0.4723872510446201 0 -0.0325 rpy=0 0 0
- joint Joint4: origin xyz=0.39129942237676174 0 0.0325 rpy=0 0 3.1416 -> xyz=0.48959223652033046 0 0.0325 rpy=0 0 3.1416

Commit message: add 3dof can train

File: dynamics/src/dynamics/urdf/single_arm_v12.urdf (robot description, URDF)
Before this commit: robot single_arm_v12, 8 links, 7 joints
Links:
- link Link2: mass 0.5043461294231942 -> 0.4420296748872608
- link Link3: mass 0.4691908056563082 -> 0.4576530992635291
Joints:
- joint Joint3: origin xyz=0.4723872510446201 0 -0.0325 rpy=0 0 0 -> xyz=0.22687587384078153 0 -0.0325 rpy=0 0 0
- joint Joint4: origin xyz=0.48959223652033046 0 0.0325 rpy=0 0 3.1416 -> xyz=0.4441365389502654 0 0.0325 rpy=0 0 3.1416

Commit message: Use virtual links, 5 dof no problem, but 4dof

File: dynamics/src/dynamics/urdf/single_arm_v12.urdf (robot description, URDF)
Before this commit: robot single_arm_v12, 8 links, 7 joints
Links:
- link Link2: mass 0.4420296748872608 -> 0.44517334347194654
- link Link3: mass 0.4576530992635291 -> 0.432690248594842
Joints:
- joint Joint3: origin xyz=0.22687587384078153 0 -0.0325 rpy=0 0 0 -> xyz=0.23926114847564672 0 -0.0325 rpy=0 0 0
- joint Joint4: origin xyz=0.4441365389502654 0 0.0325 rpy=0 0 3.1416 -> xyz=0.34578910733312096 0 0.0325 rpy=0 0 3.1416

Commit message: fixed observation & reward

File: dynamics/src/dynamics/urdf/single_arm_v12.urdf (robot description, URDF)
Before this commit: robot single_arm_v12, 8 links, 7 joints
Links:
- link Link2: mass 0.44517334347194654 -> 0.49479871700223177
- link Link3: mass 0.432690248594842 -> 0.4091523311012555
Joints:
- joint Joint3: origin xyz=0.23926114847564672 0 -0.0325 rpy=0 0 0 -> xyz=0.4347728137397521 0 -0.0325 rpy=0 0 0
- joint Joint4: origin xyz=0.34578910733312096 0 0.0325 rpy=0 0 3.1416 -> xyz=0.253055558515548 0 0.0325 rpy=0 0 3.1416

Commit message: Cancel unnecessary observations

File: dynamics/src/dynamics/urdf/single_arm_v12.urdf (robot description, URDF)
Before this commit: robot single_arm_v12, 8 links, 7 joints
Links:
- link Link2: mass 0.49479871700223177 -> 0.4846724178718292
- link Link3: mass 0.4091523311012555 -> 0.389236682260963
Joints:
- joint Joint3: origin xyz=0.4347728137397521 0 -0.0325 rpy=0 0 0 -> xyz=0.3948777063560417 0 -0.0325 rpy=0 0 0
- joint Joint4: origin xyz=0.253055558515548 0 0.0325 rpy=0 0 3.1416 -> xyz=0.17459284852992007 0 0.0325 rpy=0 0 3.1416

Commit message: learning rate & inf reward fixed

File: dynamics/src/dynamics/urdf/single_arm_v12.urdf (robot description, URDF)
Before this commit: robot single_arm_v12, 8 links, 7 joints
Links:
- link Link2: mass 0.4846724178718292 -> 0.4345456498079968
- link Link3: mass 0.389236682260963 -> 0.4530510138427058
Joints:
- joint Joint3: origin xyz=0.3948777063560417 0 -0.0325 rpy=0 0 0 -> xyz=0.19739067096906374 0 -0.0325 rpy=0 0 0
- joint Joint4: origin xyz=0.17459284852992007 0 0.0325 rpy=0 0 3.1416 -> xyz=0.4260054654111197 0 0.0325 rpy=0 0 3.1416

Commit message: fixed reward

File: dynamics/src/dynamics/urdf/single_arm_v12.urdf (robot description, URDF)
Before this commit: robot single_arm_v12, 8 links, 7 joints
Links:
- link Link2: mass 0.4345456498079968 -> 0.44070064105027873
- link Link3: mass 0.4530510138427058 -> 0.4071341231616095
Joints:
- joint Joint3: origin xyz=0.19739067096906374 0 -0.0325 rpy=0 0 0 -> xyz=0.22163981010612493 0 -0.0325 rpy=0 0 0
- joint Joint4: origin xyz=0.4260054654111197 0 0.0325 rpy=0 0 3.1416 -> xyz=0.24510432049518494 0 0.0325 rpy=0 0 3.1416

Commit message: learning rate 1e-3

File: dynamics/src/dynamics/urdf/single_arm_v12.urdf (robot description, URDF)
Before this commit: robot single_arm_v12, 8 links, 7 joints
Links:
- link Link2: mass 0.44070064105027873 -> 0.4567882906510457
- link Link3: mass 0.4071341231616095 -> 0.4357805818200342
Joints:
- joint Joint3: origin xyz=0.22163981010612493 0 -0.0325 rpy=0 0 0 -> xyz=0.2850211600059269 0 -0.0325 rpy=0 0 0
- joint Joint4: origin xyz=0.24510432049518494 0 0.0325 rpy=0 0 3.1416 -> xyz=0.3579642526950255 0 0.0325 rpy=0 0 3.1416

Commit message: fixed tested error & reward

File: dynamics/src/dynamics/urdf/single_arm_v12.urdf (robot description, URDF)
Before this commit: robot single_arm_v12, 8 links, 7 joints
Links:
- link Link2: mass 0.4567882906510457 -> 0.49560824790223124
- link Link3: mass 0.4357805818200342 -> 0.3925381331655871
- link Link6: mass 5.5581 -> 0.0173494454294496
Joints:
- joint Joint1: limit lower=-3.14 upper=3.14 effort=0 velocity=0 -> lower=-3.14 upper=3.14 effort=50 velocity=0
- joint Joint2: limit lower=-3.14 upper=3.14 effort=0 velocity=0 -> lower=-3.14 upper=3.14 effort=50 velocity=0
- joint Joint3: limit lower=-3.14 upper=3.14 effort=0 velocity=0 -> lower=-3.14 upper=3.14 effort=50 velocity=0; origin xyz=0.2850211600059269 0 -0.0325 rpy=0 0 0 -> xyz=0.43796216473264815 0 -0.0325 rpy=0 0 0
- joint Joint4: limit lower=-3.14 upper=3.14 effort=0 velocity=0 -> lower=-3.14 upper=3.14 effort=50 velocity=0; origin xyz=0.3579642526950255 0 0.0325 rpy=0 0 3.1416 -> xyz=0.18759974511353697 0 0.0325 rpy=0 0 3.1416
- joint Joint5: limit lower=-3.14 upper=3.14 effort=0 velocity=0 -> lower=-3.14 upper=3.14 effort=50 velocity=0
- joint Joint6: limit lower=-3.14 upper=3.14 effort=0 velocity=0 -> lower=-3.14 upper=3.14 effort=50 velocity=0; origin xyz=0.0346 0.068329 -0.0048371 rpy=3.1416 1.5001 -1.5708 -> xyz=0.0346 0.068329 -0.0048371 rpy=1.5708 -1.5708 0

Commit message: add C51 network

File: dynamics/src/dynamics/urdf/single_arm_v12.urdf (robot description, URDF)
Before this commit: robot single_arm_v12, 8 links, 7 joints
Links:
- link Link2: mass 0.49560824790223124 -> 0.46906182070141117
- link Link3: mass 0.3925381331655871 -> 0.3838562493205037
Joints:
- joint Joint3: origin xyz=0.43796216473264815 0 -0.0325 rpy=0 0 0 -> xyz=0.33337582472903593 0 -0.0325 rpy=0 0 0
- joint Joint4: origin xyz=0.18759974511353697 0 0.0325 rpy=0 0 3.1416 -> xyz=0.15339527908140346 0 0.0325 rpy=0 0 3.1416

Commit message: train C51

File: dynamics/src/dynamics/urdf/single_arm_v12.urdf (robot description, URDF)
Before this commit: robot single_arm_v12, 8 links, 7 joints
Links:
- link Link2: mass 0.46906182070141117 -> 0.4400797904225647
- link Link3: mass 0.3838562493205037 -> 0.39865130709256674
Joints:
- joint Joint3: origin xyz=0.33337582472903593 0 -0.0325 rpy=0 0 0 -> xyz=0.21919381259578763 0 -0.0325 rpy=0 0 0
- joint Joint4: origin xyz=0.15339527908140346 0 0.0325 rpy=0 0 3.1416 -> xyz=0.21168413205823364 0 0.0325 rpy=0 0 3.1416

Commit message: fixed compute_avg_return

File: dynamics/src/dynamics/urdf/single_arm_v12.urdf (robot description, URDF)
Before this commit: robot single_arm_v12, 8 links, 7 joints
Links:
- link Link2: mass 0.4400797904225647 -> 0.4249052659591132
- link Link3: mass 0.39865130709256674 -> 0.4650957459486376
Joints:
- joint Joint3: origin xyz=0.21919381259578763 0 -0.0325 rpy=0 0 0 -> xyz=0.15940994929388747 0 -0.0325 rpy=0 0 0
- joint Joint4: origin xyz=0.21168413205823364 0 0.0325 rpy=0 0 3.1416 -> xyz=0.4734587183611465 0 0.0325 rpy=0 0 3.1416

Commit message: fixed tb.add_scalar  input data type

File: dynamics/src/dynamics/urdf/single_arm_v12.urdf (robot description, URDF)
Before this commit: robot single_arm_v12, 8 links, 7 joints
Links:
- link Link2: mass 0.4249052659591132 -> 0.5127276082043659
- link Link3: mass 0.4650957459486376 -> 0.4586280284314029
Joints:
- joint Joint3: origin xyz=0.15940994929388747 0 -0.0325 rpy=0 0 0 -> xyz=0.5054081989450445 0 -0.0325 rpy=0 0 0
- joint Joint4: origin xyz=0.4734587183611465 0 0.0325 rpy=0 0 3.1416 -> xyz=0.4479775177287548 0 0.0325 rpy=0 0 3.1416

Commit message: add save model

File: dynamics/src/dynamics/urdf/single_arm_v12.urdf (robot description, URDF)
Before this commit: robot single_arm_v12, 8 links, 7 joints
Links:
- link Link2: mass 0.5127276082043659 -> 0.4907820562500897
- link Link3: mass 0.4586280284314029 -> 0.45044270958455973
Joints:
- joint Joint3: origin xyz=0.5054081989450445 0 -0.0325 rpy=0 0 0 -> xyz=0.41894816645577726 0 -0.0325 rpy=0 0 0
- joint Joint4: origin xyz=0.4479775177287548 0 0.0325 rpy=0 0 3.1416 -> xyz=0.4157293944579534 0 0.0325 rpy=0 0 3.1416

Commit message: add train tensorboard record & test model

File: dynamics/src/dynamics/urdf/single_arm_v12.urdf (robot description, URDF)
Before this commit: robot single_arm_v12, 8 links, 7 joints
Links:
- link Link2: mass 0.4907820562500897 -> 0.4255375306291948
- link Link3: mass 0.45044270958455973 -> 0.41112230879107936
Joints:
- joint Joint3: origin xyz=0.41894816645577726 0 -0.0325 rpy=0 0 0 -> xyz=0.16190091530061956 0 -0.0325 rpy=0 0 0
- joint Joint4: origin xyz=0.4157293944579534 0 0.0325 rpy=0 0 3.1416 -> xyz=0.26081678133054814 0 0.0325 rpy=0 0 3.1416

Commit message: add DRL general select function

File: dynamics/src/dynamics/urdf/single_arm_v12.urdf (robot description, URDF)
Before this commit: robot single_arm_v12, 8 links, 7 joints
Links:
- link Link2: mass 0.4255375306291948 -> 0.45437287587420766
- link Link3: mass 0.41112230879107936 -> 0.40193604971367575
Joints:
- joint Joint3: origin xyz=0.16190091530061956 0 -0.0325 rpy=0 0 0 -> xyz=0.2755050247765379 0 -0.0325 rpy=0 0 0
- joint Joint4: origin xyz=0.26081678133054814 0 0.0325 rpy=0 0 3.1416 -> xyz=0.22462520215463333 0 0.0325 rpy=0 0 3.1416

Commit message: 修改save model & read 的路徑

File: dynamics/src/dynamics/urdf/single_arm_v12.urdf (robot description, URDF)
Before this commit: robot single_arm_v12, 8 links, 7 joints
Links:
- link Link2: mass 0.45437287587420766 -> 0.4925777128295275
- link Link3: mass 0.40193604971367575 -> 0.42290267846547214
Joints:
- joint Joint3: origin xyz=0.2755050247765379 0 -0.0325 rpy=0 0 0 -> xyz=0.4260226080793569 0 -0.0325 rpy=0 0 0
- joint Joint4: origin xyz=0.22462520215463333 0 0.0325 rpy=0 0 3.1416 -> xyz=0.30722851195994716 0 0.0325 rpy=0 0 3.1416

Commit message: fixed 3,5 dof module of robot

File: dynamics/src/dynamics/urdf/single_arm_v12.urdf (robot description, URDF)
Before this commit: robot single_arm_v12, 8 links, 7 joints
Links:
- link Link2: mass 0.4925777128295275 -> 0.4177533484975215
- link Link3: mass 0.42290267846547214 -> 0.40010423462031297
Joints:
- joint Joint3: origin xyz=0.4260226080793569 0 -0.0325 rpy=0 0 0 -> xyz=0.1312331680774424 0 -0.0325 rpy=0 0 0
- joint Joint4: origin xyz=0.30722851195994716 0 0.0325 rpy=0 0 3.1416 -> xyz=0.21740830565427757 0 0.0325 rpy=0 0 3.1416

Commit message: fixed test i

File: dynamics/src/dynamics/urdf/single_arm_v12.urdf (robot description, URDF)
Before this commit: robot single_arm_v12, 8 links, 7 joints
Links:
- link Link2: mass 0.4177533484975215 -> 0.48570540482088276
- link Link3: mass 0.40010423462031297 -> 0.38173133347160804
Joints:
- joint Joint3: origin xyz=0.1312331680774424 0 -0.0325 rpy=0 0 0 -> xyz=0.39894741876802586 0 -0.0325 rpy=0 0 0
- joint Joint4: origin xyz=0.21740830565427757 0 0.0325 rpy=0 0 3.1416 -> xyz=0.14502363840161553 0 0.0325 rpy=0 0 3.1416

Commit message: fixed dqn& ddqn n_step_update

File: dynamics/src/dynamics/urdf/single_arm_v12.urdf (robot description, URDF)
Before this commit: robot single_arm_v12, 8 links, 7 joints
Links:
- link Link2: mass 0.48570540482088276 -> 0.44737809976472315
- link Link3: mass 0.38173133347160804 -> 0.4520035739407949
Joints:
- joint Joint3: origin xyz=0.39894741876802586 0 -0.0325 rpy=0 0 0 -> xyz=0.24794734151838949 0 -0.0325 rpy=0 0 0
- joint Joint4: origin xyz=0.14502363840161553 0 0.0325 rpy=0 0 3.1416 -> xyz=0.42187881234999847 0 0.0325 rpy=0 0 3.1416

Commit message: fixed reward && set episode  cut off

File: dynamics/src/dynamics/urdf/single_arm_v12.urdf (robot description, URDF)
Before this commit: robot single_arm_v12, 8 links, 7 joints
Links:
- link Link2: mass 0.44737809976472315 -> 0.4906387466457854
- link Link3: mass 0.4520035739407949 -> 0.3896288572289979
Joints:
- joint Joint3: origin xyz=0.24794734151838949 0 -0.0325 rpy=0 0 0 -> xyz=0.41838356215373035 0 -0.0325 rpy=0 0 0
- joint Joint4: origin xyz=0.42187881234999847 0 0.0325 rpy=0 0 3.1416 -> xyz=0.17613792049957133 0 0.0325 rpy=0 0 3.1416

Commit message: fixed num_iterations

File: dynamics/src/dynamics/urdf/single_arm_v12.urdf (robot description, URDF)
Before this commit: robot single_arm_v12, 8 links, 7 joints
Links:
- link Link2: mass 0.4906387466457854 -> 0.5082090510809976
- link Link3: mass 0.3896288572289979 -> 0.42374541437660773
Joints:
- joint Joint3: origin xyz=0.41838356215373035 0 -0.0325 rpy=0 0 0 -> xyz=0.4876062044221904 0 -0.0325 rpy=0 0 0
- joint Joint4: origin xyz=0.17613792049957133 0 0.0325 rpy=0 0 3.1416 -> xyz=0.31054868213969683 0 0.0325 rpy=0 0 3.1416

Commit message: fixed read urdf error

File: dynamics/src/dynamics/urdf/single_arm_v12.urdf (robot description, URDF)
Before this commit: robot single_arm_v12, 8 links, 7 joints
Links:
- link Link2: mass 0.5082090510809976 -> 0.45460603315811254
- link Link3: mass 0.42374541437660773 -> 0.39113204278905295
Joints:
- joint Joint3: origin xyz=0.4876062044221904 0 -0.0325 rpy=0 0 0 -> xyz=0.27642360665515836 0 -0.0325 rpy=0 0 0
- joint Joint4: origin xyz=0.31054868213969683 0 0.0325 rpy=0 0 3.1416 -> xyz=0.18206009826033595 0 0.0325 rpy=0 0 3.1416

Commit message: fixed Q value max & min

File: dynamics/src/dynamics/urdf/single_arm_v12.urdf (robot description, URDF)
Before this commit: robot single_arm_v12, 8 links, 7 joints
Links:
- link Link2: mass 0.45460603315811254 -> 0.43410325189126703
- link Link3: mass 0.39113204278905295 -> 0.42648924775719305
Joints:
- joint Joint3: origin xyz=0.27642360665515836 0 -0.0325 rpy=0 0 0 -> xyz=0.19564773288606027 0 -0.0325 rpy=0 0 0
- joint Joint4: origin xyz=0.18206009826033595 0 0.0325 rpy=0 0 3.1416 -> xyz=0.32135870417393697 0 0.0325 rpy=0 0 3.1416
