Commit message: add power cal & reward

File: dynamics/src/dynamics/urdf/single_arm_v12.urdf (robot description, URDF)
Before this commit: robot single_arm_v12, 8 links, 7 joints
Links:
- link Link2: mass 0.43410325189126703 -> 0.4096022585637529
- link Link3: mass 0.42648924775719305 -> 0.4458493238227684
Joints:
- joint Joint3: origin xyz=0.19564773288606027 0 -0.0325 rpy=0 0 0 -> xyz=0.09911989510235761 0 -0.0325 rpy=0 0 0
- joint Joint4: origin xyz=0.32135870417393697 0 0.0325 rpy=0 0 3.1416 -> xyz=0.39763259541466117 0 0.0325 rpy=0 0 3.1416

Commit message: add pybullet test code

File: dynamics/src/dynamics/urdf/single_arm_v12.urdf (robot description, URDF)
Before this commit: robot single_arm_v12, 8 links, 7 joints
Links:
- link Link2: mass 0.4096022585637529 -> 0.42078380873388094
- link Link3: mass 0.4458493238227684 -> 0.38641553425368397
Joints:
- joint Joint3: origin xyz=0.09911989510235761 0 -0.0325 rpy=0 0 0 -> xyz=0.1431724298940955 0 -0.0325 rpy=0 0 0
- joint Joint4: origin xyz=0.39763259541466117 0 0.0325 rpy=0 0 3.1416 -> xyz=0.16347822606912318 0 0.0325 rpy=0 0 3.1416

Commit message: add param for server train

File: dynamics/src/dynamics/urdf/single_arm_v12.urdf (robot description, URDF)
Before this commit: robot single_arm_v12, 8 links, 7 joints
Links:
- link Link2: mass 0.42078380873388094 -> 0.45259942878739007
- link Link3: mass 0.38641553425368397 -> 0.45821014701394563
Joints:
- joint Joint3: origin xyz=0.1431724298940955 0 -0.0325 rpy=0 0 0 -> xyz=0.2685180830462175 0 -0.0325 rpy=0 0 0
- joint Joint4: origin xyz=0.16347822606912318 0 0.0325 rpy=0 0 3.1416 -> xyz=0.44633116873308487 0 0.0325 rpy=0 0 3.1416

Commit message: fixed random point

File: dynamics/src/dynamics/urdf/single_arm_v12.urdf (robot description, URDF)
Before this commit: robot single_arm_v12, 8 links, 7 joints
Links:
- link Link2: mass 0.45259942878739007 -> 0.45028638757544864
- link Link3: mass 0.45821014701394563 -> 0.4151523163710768
Joints:
- joint Joint3: origin xyz=0.2685180830462175 0 -0.0325 rpy=0 0 0 -> xyz=0.25940527427521276 0 -0.0325 rpy=0 0 0
- joint Joint4: origin xyz=0.44633116873308487 0 0.0325 rpy=0 0 3.1416 -> xyz=0.27669401026368157 0 0.0325 rpy=0 0 3.1416

Commit message: add power consumption train data

File: dynamics/src/dynamics/urdf/single_arm_v12.urdf (robot description, URDF)
Before this commit: robot single_arm_v12, 8 links, 7 joints
Links:
- link Link2: mass 0.42078380873388094 -> 0.5252553866184609
- link Link3: mass 0.38641553425368397 -> 0.42916693433405645
Joints:
- joint Joint3: origin xyz=0.1431724298940955 0 -0.0325 rpy=0 0 0 -> xyz=0.5547645391709706 0 -0.0325 rpy=0 0 0
- joint Joint4: origin xyz=0.16347822606912318 0 0.0325 rpy=0 0 3.1416 -> xyz=0.3319081242303791 0 0.0325 rpy=0 0 3.1416

Commit message: add c51 test result

File: dynamics/src/dynamics/urdf/single_arm_v12.urdf (robot description, URDF)
Before this commit: robot single_arm_v12, 8 links, 7 joints
Links:
- link Link2: mass 0.5252553866184609 -> 0.5187783113950207
- link Link3: mass 0.42916693433405645 -> 0.525960218562696
Joints:
- joint Joint3: origin xyz=0.5547645391709706 0 -0.0325 rpy=0 0 0 -> xyz=0.5292464690207715 0 -0.0325 rpy=0 0 0
- joint Joint4: origin xyz=0.3319081242303791 0 0.0325 rpy=0 0 3.1416 -> xyz=0.7132496235654634 0 0.0325 rpy=0 0 3.1416

Commit message: server train tf agent error fixed

File: dynamics/src/dynamics/urdf/single_arm_v12.urdf (robot description, URDF)
Before this commit: robot single_arm_v12, 8 links, 7 joints
Links:
- link Link2: mass 0.45028638757544864 -> 0.4445264046156597
- link Link3: mass 0.4151523163710768 -> 0.45870870188912355
Joints:
- joint Joint3: origin xyz=0.25940527427521276 0 -0.0325 rpy=0 0 0 -> xyz=0.2367123698142729 0 -0.0325 rpy=0 0 0
- joint Joint4: origin xyz=0.27669401026368157 0 0.0325 rpy=0 0 3.1416 -> xyz=0.44829535111532604 0 0.0325 rpy=0 0 3.1416

Commit message: set test point show & obstacles

File: dynamics/src/dynamics/urdf/single_arm_v12.urdf (robot description, URDF)
Before this commit: robot single_arm_v12, 8 links, 7 joints
Links:
- link Link2: mass 0.5605965604710196 -> 0.43876148089988687
- link Link3: mass 0.5210742192987424 -> 0.3992391278891867
Joints:
- joint Joint3: origin xyz=0.694 0 -0.0325 rpy=0 0 0 -> xyz=0.214 0 -0.0325 rpy=0 0 0
- joint Joint4: origin xyz=0.694 0 0.0325 rpy=0 0 3.1416 -> xyz=0.214 0 0.0325 rpy=0 0 3.1416

File: dynamics/src/dynamics/urdf/single_arm_v12_motion.urdf (robot description, URDF)
Before this commit: robot single_arm_v12, 8 links, 7 joints
Links:
- link Link2: mass 0.5605965604710196 -> 0.43876148089988687
- link Link3: mass 0.5210742192987424 -> 0.3992391278891867
Joints:
- joint Joint3: origin xyz=0.694 0 -0.0325 rpy=0 0 0 -> xyz=0.214 0 -0.0325 rpy=0 0 0
- joint Joint4: origin xyz=0.694 0 0.0325 rpy=0 0 3.1416 -> xyz=0.214 0 0.0325 rpy=0 0 3.1416

Commit message: update motion reward

File: dynamics/src/dynamics/urdf/single_arm_v12.urdf (robot description, URDF)
Before this commit: robot single_arm_v12, 8 links, 7 joints
Links:
- link Link2: mass 0.43876148089988687 -> 0.46683162511997356
- link Link3: mass 0.3992391278891867 -> 0.41959557208320725
Joints:
- joint Joint3: origin xyz=0.214 0 -0.0325 rpy=0 0 0 -> xyz=0.3245894071975805 0 -0.0325 rpy=0 0 0
- joint Joint4: origin xyz=0.214 0 0.0325 rpy=0 0 3.1416 -> xyz=0.2941993341990755 0 0.0325 rpy=0 0 3.1416

File: dynamics/src/dynamics/urdf/single_arm_v12_motion.urdf (robot description, URDF)
Before this commit: robot single_arm_v12, 8 links, 7 joints
Links:
- link Link2: mass 0.43876148089988687 -> 0.46683162511997356
- link Link3: mass 0.3992391278891867 -> 0.41959557208320725
Joints:
- joint Joint3: origin xyz=0.214 0 -0.0325 rpy=0 0 0 -> xyz=0.3245894071975805 0 -0.0325 rpy=0 0 0
- joint Joint4: origin xyz=0.214 0 0.0325 rpy=0 0 3.1416 -> xyz=0.2941993341990755 0 0.0325 rpy=0 0 3.1416

Commit message: test pybullet robot angle

File: dynamics/src/dynamics/urdf/single_arm_v12.urdf (robot description, URDF)
Before this commit: robot single_arm_v12, 8 links, 7 joints
Links:
- link Link2: mass 0.46683162511997356 -> 0.43876148089988687
- link Link3: mass 0.41959557208320725 -> 0.3992391278891867
Joints:
- joint Joint3: origin xyz=0.3245894071975805 0 -0.0325 rpy=0 0 0 -> xyz=0.214 0 -0.0325 rpy=0 0 0
- joint Joint4: origin xyz=0.2941993341990755 0 0.0325 rpy=0 0 3.1416 -> xyz=0.214 0 0.0325 rpy=0 0 3.1416

File: dynamics/src/dynamics/urdf/single_arm_v12_motion.urdf (robot description, URDF)
Before this commit: robot single_arm_v12, 8 links, 7 joints
Links:
- link Link2: mass 0.46683162511997356 -> 0.43876148089988687
- link Link3: mass 0.41959557208320725 -> 0.3992391278891867
Joints:
- joint Joint3: origin xyz=0.3245894071975805 0 -0.0325 rpy=0 0 0 -> xyz=0.214 0 -0.0325 rpy=0 0 0
- joint Joint4: origin xyz=0.2941993341990755 0 0.0325 rpy=0 0 3.1416 -> xyz=0.214 0 0.0325 rpy=0 0 3.1416

Commit message: server train case 3

File: dynamics/src/dynamics/urdf/single_arm_v12.urdf (robot description, URDF)
Before this commit: robot single_arm_v12, 8 links, 7 joints
Links:
- link Link2: mass 0.43876148089988687 -> 0.4218174588914997
- link Link3: mass 0.3992391278891867 -> 0.44025081972857294
Joints:
- joint Joint3: origin xyz=0.214 0 -0.0325 rpy=0 0 0 -> xyz=0.1472447551833592 0 -0.0325 rpy=0 0 0
- joint Joint4: origin xyz=0.214 0 0.0325 rpy=0 0 3.1416 -> xyz=0.37557587978270623 0 0.0325 rpy=0 0 3.1416

File: dynamics/src/dynamics/urdf/single_arm_v12_motion.urdf (robot description, URDF)
Before this commit: robot single_arm_v12, 8 links, 7 joints
Links:
- link Link2: mass 0.43876148089988687 -> 0.4218174588914997
- link Link3: mass 0.3992391278891867 -> 0.44025081972857294
Joints:
- joint Joint3: origin xyz=0.214 0 -0.0325 rpy=0 0 0 -> xyz=0.1472447551833592 0 -0.0325 rpy=0 0 0
- joint Joint4: origin xyz=0.214 0 0.0325 rpy=0 0 3.1416 -> xyz=0.37557587978270623 0 0.0325 rpy=0 0 3.1416

Commit message: fixed train & test config input

File: dynamics/src/dynamics/urdf/single_arm_v12.urdf (robot description, URDF)
Before this commit: robot single_arm_v12, 8 links, 7 joints
Links:
- link Link2: mass 0.4218174588914997 -> 0.49805864020239143
- link Link3: mass 0.44025081972857294 -> 0.4719939873754139
Joints:
- joint Joint3: origin xyz=0.1472447551833592 0 -0.0325 rpy=0 0 0 -> xyz=0.4476161027299568 0 -0.0325 rpy=0 0 0
- joint Joint4: origin xyz=0.37557587978270623 0 0.0325 rpy=0 0 3.1416 -> xyz=0.5006360762680077 0 0.0325 rpy=0 0 3.1416

File: dynamics/src/dynamics/urdf/single_arm_v12_motion.urdf (robot description, URDF)
Before this commit: robot single_arm_v12, 8 links, 7 joints
Links:
- link Link2: mass 0.4218174588914997 -> 0.49805864020239143
- link Link3: mass 0.44025081972857294 -> 0.4719939873754139
Joints:
- joint Joint3: origin xyz=0.1472447551833592 0 -0.0325 rpy=0 0 0 -> xyz=0.4476161027299568 0 -0.0325 rpy=0 0 0
- joint Joint4: origin xyz=0.37557587978270623 0 0.0325 rpy=0 0 3.1416 -> xyz=0.5006360762680077 0 0.0325 rpy=0 0 3.1416

Commit message: test model v1

File: dynamics/src/dynamics/urdf/single_arm_v12.urdf (robot description, URDF)
Before this commit: robot single_arm_v12, 8 links, 7 joints
Links:
- link Link2: mass 0.49805864020239143 -> 0.5129384837812501
- link Link3: mass 0.4719939873754139 -> 0.5202631601042224
Joints:
- joint Joint3: origin xyz=0.4476161027299568 0 -0.0325 rpy=0 0 0 -> xyz=0.5062389964235761 0 -0.0325 rpy=0 0 0
- joint Joint4: origin xyz=0.5006360762680077 0 0.0325 rpy=0 0 3.1416 -> xyz=0.690804628216177 0 0.0325 rpy=0 0 3.1416

File: dynamics/src/dynamics/urdf/single_arm_v12_motion.urdf (robot description, URDF)
Before this commit: robot single_arm_v12, 8 links, 7 joints
Links:
- link Link2: mass 0.49805864020239143 -> 0.5129384837812501
- link Link3: mass 0.4719939873754139 -> 0.5202631601042224
Joints:
- joint Joint3: origin xyz=0.4476161027299568 0 -0.0325 rpy=0 0 0 -> xyz=0.5062389964235761 0 -0.0325 rpy=0 0 0
- joint Joint4: origin xyz=0.5006360762680077 0 0.0325 rpy=0 0 3.1416 -> xyz=0.690804628216177 0 0.0325 rpy=0 0 3.1416

Commit message: test model v2

File: dynamics/src/dynamics/urdf/single_arm_v12.urdf (robot description, URDF)
Before this commit: robot single_arm_v12, 8 links, 7 joints
Links:
- link Link2: mass 0.5129384837812501 -> 0.4799165704982845
- link Link3: mass 0.5202631601042224 -> 0.4707959871255701
Joints:
- joint Joint3: origin xyz=0.5062389964235761 0 -0.0325 rpy=0 0 0 -> xyz=0.37614084709237905 0 -0.0325 rpy=0 0 0
- joint Joint4: origin xyz=0.690804628216177 0 0.0325 rpy=0 0 3.1416 -> xyz=0.4959162528306694 0 0.0325 rpy=0 0 3.1416

File: dynamics/src/dynamics/urdf/single_arm_v12_motion.urdf (robot description, URDF)
Before this commit: robot single_arm_v12, 8 links, 7 joints
Links:
- link Link2: mass 0.5129384837812501 -> 0.4799165704982845
- link Link3: mass 0.5202631601042224 -> 0.4707959871255701
Joints:
- joint Joint3: origin xyz=0.5062389964235761 0 -0.0325 rpy=0 0 0 -> xyz=0.37614084709237905 0 -0.0325 rpy=0 0 0
- joint Joint4: origin xyz=0.690804628216177 0 0.0325 rpy=0 0 3.1416 -> xyz=0.4959162528306694 0 0.0325 rpy=0 0 3.1416

Commit message: test model v3

File: dynamics/src/dynamics/urdf/single_arm_v12.urdf (robot description, URDF)
Before this commit: robot single_arm_v12, 8 links, 7 joints
Links:
- link Link2: mass 0.4799165704982845 -> 0.46814901217779514
- link Link3: mass 0.4707959871255701 -> 0.47859817520534687
Joints:
- joint Joint3: origin xyz=0.37614084709237905 0 -0.0325 rpy=0 0 0 -> xyz=0.3297795855105938 0 -0.0325 rpy=0 0 0
- joint Joint4: origin xyz=0.4959162528306694 0 0.0325 rpy=0 0 3.1416 -> xyz=0.5266549360373299 0 0.0325 rpy=0 0 3.1416

File: dynamics/src/dynamics/urdf/single_arm_v12_motion.urdf (robot description, URDF)
Before this commit: robot single_arm_v12, 8 links, 7 joints
Links:
- link Link2: mass 0.4799165704982845 -> 0.46814901217779514
- link Link3: mass 0.4707959871255701 -> 0.47859817520534687
Joints:
- joint Joint3: origin xyz=0.37614084709237905 0 -0.0325 rpy=0 0 0 -> xyz=0.3297795855105938 0 -0.0325 rpy=0 0 0
- joint Joint4: origin xyz=0.4959162528306694 0 0.0325 rpy=0 0 3.1416 -> xyz=0.5266549360373299 0 0.0325 rpy=0 0 3.1416

Commit message: test model v4

File: dynamics/src/dynamics/urdf/single_arm_v12.urdf (robot description, URDF)
Before this commit: robot single_arm_v12, 8 links, 7 joints
Links:
- link Link2: mass 0.46814901217779514 -> 0.4772136711923573
- link Link3: mass 0.47859817520534687 -> 0.4012562983536959
Joints:
- joint Joint3: origin xyz=0.3297795855105938 0 -0.0325 rpy=0 0 0 -> xyz=0.36549209411079164 0 -0.0325 rpy=0 0 0
- joint Joint4: origin xyz=0.5266549360373299 0 0.0325 rpy=0 0 3.1416 -> xyz=0.2219471506260018 0 0.0325 rpy=0 0 3.1416

File: dynamics/src/dynamics/urdf/single_arm_v12_motion.urdf (robot description, URDF)
Before this commit: robot single_arm_v12, 8 links, 7 joints
Links:
- link Link2: mass 0.46814901217779514 -> 0.4772136711923573
- link Link3: mass 0.47859817520534687 -> 0.4012562983536959
Joints:
- joint Joint3: origin xyz=0.3297795855105938 0 -0.0325 rpy=0 0 0 -> xyz=0.36549209411079164 0 -0.0325 rpy=0 0 0
- joint Joint4: origin xyz=0.5266549360373299 0 0.0325 rpy=0 0 3.1416 -> xyz=0.2219471506260018 0 0.0325 rpy=0 0 3.1416

Commit message: todo record episode step reward

File: dynamics/src/dynamics/urdf/single_arm_v12.urdf (robot description, URDF)
Before this commit: robot single_arm_v12, 8 links, 7 joints
Links:
- link Link2: mass 0.4772136711923573 -> 0.4476704145464963
- link Link3: mass 0.4012562983536959 -> 0.43743843270024985
Joints:
- joint Joint3: origin xyz=0.36549209411079164 0 -0.0325 rpy=0 0 0 -> xyz=0.2490989892683234 0 -0.0325 rpy=0 0 0
- joint Joint4: origin xyz=0.2219471506260018 0 0.0325 rpy=0 0 3.1416 -> xyz=0.36449577340303313 0 0.0325 rpy=0 0 3.1416

File: dynamics/src/dynamics/urdf/single_arm_v12_motion.urdf (robot description, URDF)
Before this commit: robot single_arm_v12, 8 links, 7 joints
Links:
- link Link2: mass 0.4772136711923573 -> 0.4476704145464963
- link Link3: mass 0.4012562983536959 -> 0.43743843270024985
Joints:
- joint Joint3: origin xyz=0.36549209411079164 0 -0.0325 rpy=0 0 0 -> xyz=0.2490989892683234 0 -0.0325 rpy=0 0 0
- joint Joint4: origin xyz=0.2219471506260018 0 0.0325 rpy=0 0 3.1416 -> xyz=0.36449577340303313 0 0.0325 rpy=0 0 3.1416

Commit message: catch manipulability plot view

File: dynamics/src/dynamics/urdf/single_arm_v12.urdf (robot description, URDF)
Before this commit: robot single_arm_v12, 8 links, 7 joints
Links:
- link Link2: mass 0.4476704145464963 -> 0.43876148089988687
- link Link3: mass 0.43743843270024985 -> 0.3992391278891867
Joints:
- joint Joint3: origin xyz=0.2490989892683234 0 -0.0325 rpy=0 0 0 -> xyz=0.214 0 -0.0325 rpy=0 0 0
- joint Joint4: origin xyz=0.36449577340303313 0 0.0325 rpy=0 0 3.1416 -> xyz=0.214 0 0.0325 rpy=0 0 3.1416

File: dynamics/src/dynamics/urdf/single_arm_v12_motion.urdf (robot description, URDF)
Before this commit: robot single_arm_v12, 8 links, 7 joints
Links:
- link Link2: mass 0.4476704145464963 -> 0.43876148089988687
- link Link3: mass 0.43743843270024985 -> 0.3992391278891867
Joints:
- joint Joint3: origin xyz=0.2490989892683234 0 -0.0325 rpy=0 0 0 -> xyz=0.214 0 -0.0325 rpy=0 0 0
- joint Joint4: origin xyz=0.36449577340303313 0 0.0325 rpy=0 0 3.1416 -> xyz=0.214 0 0.0325 rpy=0 0 3.1416

Commit message: test model v5 excel traj

File: dynamics/src/dynamics/urdf/single_arm_v12.urdf (robot description, URDF)
Before this commit: robot single_arm_v12, 8 links, 7 joints
Links:
- link Link2: mass 0.43876148089988687 -> 0.5456394086042491
- link Link3: mass 0.3992391278891867 -> 0.4401915227539354
Joints:
- joint Joint3: origin xyz=0.214 0 -0.0325 rpy=0 0 0 -> xyz=0.6350725308234552 0 -0.0325 rpy=0 0 0
- joint Joint4: origin xyz=0.214 0 0.0325 rpy=0 0 3.1416 -> xyz=0.37534226443021024 0 0.0325 rpy=0 0 3.1416

File: dynamics/src/dynamics/urdf/single_arm_v12_motion.urdf (robot description, URDF)
Before this commit: robot single_arm_v12, 8 links, 7 joints
Links:
- link Link2: mass 0.43876148089988687 -> 0.5456394086042491
- link Link3: mass 0.3992391278891867 -> 0.4401915227539354
Joints:
- joint Joint3: origin xyz=0.214 0 -0.0325 rpy=0 0 0 -> xyz=0.6350725308234552 0 -0.0325 rpy=0 0 0
- joint Joint4: origin xyz=0.214 0 0.0325 rpy=0 0 3.1416 -> xyz=0.37534226443021024 0 0.0325 rpy=0 0 3.1416

Commit message: fixed case3 obstacle random problem

File: dynamics/src/dynamics/urdf/single_arm_v12.urdf (robot description, URDF)
Before this commit: robot single_arm_v12, 8 links, 7 joints
Links:
- link Link2: mass 0.5456394086042491 -> 0.5018490197691595
- link Link3: mass 0.4401915227539354 -> 0.454041506783325
Joints:
- joint Joint3: origin xyz=0.6350725308234552 0 -0.0325 rpy=0 0 0 -> xyz=0.4625492582583405 0 -0.0325 rpy=0 0 0
- joint Joint4: origin xyz=0.37534226443021024 0 0.0325 rpy=0 0 3.1416 -> xyz=0.4299077615886555 0 0.0325 rpy=0 0 3.1416

File: dynamics/src/dynamics/urdf/single_arm_v12_motion.urdf (robot description, URDF)
Before this commit: robot single_arm_v12, 8 links, 7 joints
Links:
- link Link2: mass 0.5456394086042491 -> 0.5018490197691595
- link Link3: mass 0.4401915227539354 -> 0.454041506783325
Joints:
- joint Joint3: origin xyz=0.6350725308234552 0 -0.0325 rpy=0 0 0 -> xyz=0.4625492582583405 0 -0.0325 rpy=0 0 0
- joint Joint4: origin xyz=0.37534226443021024 0 0.0325 rpy=0 0 3.1416 -> xyz=0.4299077615886555 0 0.0325 rpy=0 0 3.1416

Commit message: case2 add 3,5 dof

File: dynamics/src/dynamics/urdf/single_arm_v12.urdf (robot description, URDF)
Before this commit: robot single_arm_v12, 8 links, 7 joints
Links:
- link Link2: mass 0.5018490197691595 -> 0.4452699243594632
- link Link3: mass 0.454041506783325 -> 0.4031738824185237
Joints:
- joint Joint3: origin xyz=0.4625492582583405 0 -0.0325 rpy=0 0 0 -> xyz=0.23964165322166248 0 -0.0325 rpy=0 0 0
- joint Joint4: origin xyz=0.4299077615886555 0 0.0325 rpy=0 0 3.1416 -> xyz=0.22950195557150987 0 0.0325 rpy=0 0 3.1416

File: dynamics/src/dynamics/urdf/single_arm_v12_motion.urdf (robot description, URDF)
Before this commit: robot single_arm_v12, 8 links, 7 joints
Links:
- link Link2: mass 0.5018490197691595 -> 0.4452699243594632
- link Link3: mass 0.454041506783325 -> 0.4031738824185237
Joints:
- joint Joint3: origin xyz=0.4625492582583405 0 -0.0325 rpy=0 0 0 -> xyz=0.23964165322166248 0 -0.0325 rpy=0 0 0
- joint Joint4: origin xyz=0.4299077615886555 0 0.0325 rpy=0 0 3.1416 -> xyz=0.22950195557150987 0 0.0325 rpy=0 0 3.1416

Commit message: server train case3

File: dynamics/src/dynamics/urdf/single_arm_v12.urdf (robot description, URDF)
Before this commit: robot single_arm_v12, 8 links, 7 joints
Links:
- link Link2: mass 0.5018490197691595 -> 0.4367226205713059
- link Link3: mass 0.454041506783325 -> 0.43872509144247096
Joints:
- joint Joint3: origin xyz=0.4625492582583405 0 -0.0325 rpy=0 0 0 -> xyz=0.20596739591615326 0 -0.0325 rpy=0 0 0
- joint Joint4: origin xyz=0.4299077615886555 0 0.0325 rpy=0 0 3.1416 -> xyz=0.36956488928024817 0 0.0325 rpy=0 0 3.1416

File: dynamics/src/dynamics/urdf/single_arm_v12_motion.urdf (robot description, URDF)
Before this commit: robot single_arm_v12, 8 links, 7 joints
Links:
- link Link2: mass 0.5018490197691595 -> 0.4367226205713059
- link Link3: mass 0.454041506783325 -> 0.43872509144247096
Joints:
- joint Joint3: origin xyz=0.4625492582583405 0 -0.0325 rpy=0 0 0 -> xyz=0.20596739591615326 0 -0.0325 rpy=0 0 0
- joint Joint4: origin xyz=0.4299077615886555 0 0.0325 rpy=0 0 3.1416 -> xyz=0.36956488928024817 0 0.0325 rpy=0 0 3.1416

Commit message: Added specified armlength & Test config motor

File: dynamics/src/dynamics/urdf/single_arm_v12.urdf (robot description, URDF)
Before this commit: robot single_arm_v12, 8 links, 7 joints
Links:
- link Link2: mass 0.4452699243594632 -> 0.4533693171572542
- link Link3: mass 0.4031738824185237 -> 0.3960830069394972
Joints:
- joint Joint3: origin xyz=0.23964165322166248 0 -0.0325 rpy=0 0 0 -> xyz=0.27155125230121047 0 -0.0325 rpy=0 0 0
- joint Joint4: origin xyz=0.22950195557150987 0 0.0325 rpy=0 0 3.1416 -> xyz=0.20156566734325823 0 0.0325 rpy=0 0 3.1416

File: dynamics/src/dynamics/urdf/single_arm_v12_motion.urdf (robot description, URDF)
Before this commit: robot single_arm_v12, 8 links, 7 joints
Links:
- link Link2: mass 0.4452699243594632 -> 0.4533693171572542
- link Link3: mass 0.4031738824185237 -> 0.3960830069394972
Joints:
- joint Joint3: origin xyz=0.23964165322166248 0 -0.0325 rpy=0 0 0 -> xyz=0.27155125230121047 0 -0.0325 rpy=0 0 0
- joint Joint4: origin xyz=0.22950195557150987 0 0.0325 rpy=0 0 3.1416 -> xyz=0.20156566734325823 0 0.0325 rpy=0 0 3.1416

Commit message: add test xlsx & origin design arm legth test

File: dynamics/src/dynamics/urdf/single_arm_v12.urdf (robot description, URDF)
Before this commit: robot single_arm_v12, 8 links, 7 joints
Links:
- link Link2: mass 0.4533693171572542 -> 0.5138042752232314
- link Link3: mass 0.3960830069394972 -> 0.46633726625192845
Joints:
- joint Joint3: origin xyz=0.27155125230121047 0 -0.0325 rpy=0 0 0 -> xyz=0.5096499999999999 0 -0.0325 rpy=0 0 0
- joint Joint4: origin xyz=0.20156566734325823 0 0.0325 rpy=0 0 3.1416 -> xyz=0.47835000000000005 0 0.0325 rpy=0 0 3.1416

File: dynamics/src/dynamics/urdf/single_arm_v12_motion.urdf (robot description, URDF)
Before this commit: robot single_arm_v12, 8 links, 7 joints
Links:
- link Link2: mass 0.4533693171572542 -> 0.5138042752232314
- link Link3: mass 0.3960830069394972 -> 0.46633726625192845
Joints:
- joint Joint3: origin xyz=0.27155125230121047 0 -0.0325 rpy=0 0 0 -> xyz=0.5096499999999999 0 -0.0325 rpy=0 0 0
- joint Joint4: origin xyz=0.20156566734325823 0 0.0325 rpy=0 0 3.1416 -> xyz=0.47835000000000005 0 0.0325 rpy=0 0 3.1416

Commit message: train case 2 & 5 dof

File: dynamics/src/dynamics/urdf/single_arm_v12.urdf (robot description, URDF)
Before this commit: robot single_arm_v12, 8 links, 7 joints
Links:
- link Link2: mass 0.4452699243594632 -> 0.49099218860259525
- link Link3: mass 0.4031738824185237 -> 0.43995216890701616
Joints:
- joint Joint3: origin xyz=0.23964165322166248 0 -0.0325 rpy=0 0 0 -> xyz=0.4197760358145669 0 -0.0325 rpy=0 0 0
- joint Joint4: origin xyz=0.22950195557150987 0 0.0325 rpy=0 0 3.1416 -> xyz=0.3743992697216084 0 0.0325 rpy=0 0 3.1416

File: dynamics/src/dynamics/urdf/single_arm_v12_motion.urdf (robot description, URDF)
Before this commit: robot single_arm_v12, 8 links, 7 joints
Links:
- link Link2: mass 0.4452699243594632 -> 0.49099218860259525
- link Link3: mass 0.4031738824185237 -> 0.43995216890701616
Joints:
- joint Joint3: origin xyz=0.23964165322166248 0 -0.0325 rpy=0 0 0 -> xyz=0.4197760358145669 0 -0.0325 rpy=0 0 0
- joint Joint4: origin xyz=0.22950195557150987 0 0.0325 rpy=0 0 3.1416 -> xyz=0.3743992697216084 0 0.0325 rpy=0 0 3.1416
