Commit message: fixed model file location & case1 action fixed

File: dynamics/src/dynamics/urdf/single_arm_v12.urdf (robot description, URDF)
Before this commit: robot single_arm_v12, 8 links, 7 joints
Links:
- link Link2: mass 0.43876148089988687 -> 0.4740402835730256
- link Link3: mass 0.3992391278891867 -> 0.4834713345738982
Joints:
- joint Joint3: origin xyz=0.214 0 -0.0325 rpy=0 0 0 -> xyz=0.35298973384935395 0 -0.0325 rpy=0 0 0
- joint Joint4: origin xyz=0.214 0 0.0325 rpy=0 0 3.1416 -> xyz=0.5458539736039499 0 0.0325 rpy=0 0 3.1416

File: dynamics/src/dynamics/urdf/single_arm_v12_motion.urdf (robot description, URDF)
Before this commit: robot single_arm_v12, 8 links, 7 joints
Links:
- link Link2: mass 0.43876148089988687 -> 0.4740402835730256
- link Link3: mass 0.3992391278891867 -> 0.4834713345738982
Joints:
- joint Joint3: origin xyz=0.214 0 -0.0325 rpy=0 0 0 -> xyz=0.35298973384935395 0 -0.0325 rpy=0 0 0
- joint Joint4: origin xyz=0.214 0 0.0325 rpy=0 0 3.1416 -> xyz=0.5458539736039499 0 0.0325 rpy=0 0 3.1416

Commit message: case2 train fixed arm length

File: dynamics/src/dynamics/urdf/single_arm_v12.urdf (robot description, URDF)
Before this commit: robot single_arm_v12, 8 links, 7 joints
Links:
- link Link2: mass 0.5138042752232314 -> 0.47548096937081674
- link Link3: mass 0.46633726625192845 -> 0.5046605758281271
Joints:
- joint Joint3: origin xyz=0.5096499999999999 0 -0.0325 rpy=0 0 0 -> xyz=0.3586656786213686 0 -0.0325 rpy=0 0 0
- joint Joint4: origin xyz=0.47835000000000005 0 0.0325 rpy=0 0 3.1416 -> xyz=0.6293343213786313 0 0.0325 rpy=0 0 3.1416

File: dynamics/src/dynamics/urdf/single_arm_v12_motion.urdf (robot description, URDF)
Before this commit: robot single_arm_v12, 8 links, 7 joints
Links:
- link Link2: mass 0.5138042752232314 -> 0.47548096937081674
- link Link3: mass 0.46633726625192845 -> 0.5046605758281271
Joints:
- joint Joint3: origin xyz=0.5096499999999999 0 -0.0325 rpy=0 0 0 -> xyz=0.3586656786213686 0 -0.0325 rpy=0 0 0
- joint Joint4: origin xyz=0.47835000000000005 0 0.0325 rpy=0 0 3.1416 -> xyz=0.6293343213786313 0 0.0325 rpy=0 0 3.1416

Commit message: fixed & test model

File: dynamics/src/dynamics/urdf/single_arm_v12.urdf (robot description, URDF)
Before this commit: robot single_arm_v12, 8 links, 7 joints
Links:
- link Link2: mass 0.4740402835730256 -> 0.5706947485678016
- link Link3: mass 0.4834713345738982 -> 0.4094467873794471
Joints:
- joint Joint3: origin xyz=0.35298973384935395 0 -0.0325 rpy=0 0 0 -> xyz=0.7337843568824151 0 -0.0325 rpy=0 0 0
- joint Joint4: origin xyz=0.5458539736039499 0 0.0325 rpy=0 0 3.1416 -> xyz=0.2542156431175849 0 0.0325 rpy=0 0 3.1416

File: dynamics/src/dynamics/urdf/single_arm_v12_motion.urdf (robot description, URDF)
Before this commit: robot single_arm_v12, 8 links, 7 joints
Links:
- link Link2: mass 0.4740402835730256 -> 0.5706947485678016
- link Link3: mass 0.4834713345738982 -> 0.4094467873794471
Joints:
- joint Joint3: origin xyz=0.35298973384935395 0 -0.0325 rpy=0 0 0 -> xyz=0.7337843568824151 0 -0.0325 rpy=0 0 0
- joint Joint4: origin xyz=0.5458539736039499 0 0.0325 rpy=0 0 3.1416 -> xyz=0.2542156431175849 0 0.0325 rpy=0 0 3.1416

Commit message: Fixed no add payload set

File: dynamics/src/dynamics/urdf/single_arm_v12.urdf (robot description, URDF)
Before this commit: robot single_arm_v12, 8 links, 7 joints
Links:
- link Link2: mass 0.5706947485678016 -> 0.5138042752232314
- link Link3: mass 0.4094467873794471 -> 0.46633726625192845
Joints:
- joint Joint3: origin xyz=0.7337843568824151 0 -0.0325 rpy=0 0 0 -> xyz=0.5096499999999999 0 -0.0325 rpy=0 0 0
- joint Joint4: origin xyz=0.2542156431175849 0 0.0325 rpy=0 0 3.1416 -> xyz=0.47835000000000005 0 0.0325 rpy=0 0 3.1416

File: dynamics/src/dynamics/urdf/single_arm_v12_motion.urdf (robot description, URDF)
Before this commit: robot single_arm_v12, 8 links, 7 joints
Links:
- link Link2: mass 0.5706947485678016 -> 0.5138042752232314
- link Link3: mass 0.4094467873794471 -> 0.46633726625192845
Joints:
- joint Joint3: origin xyz=0.7337843568824151 0 -0.0325 rpy=0 0 0 -> xyz=0.5096499999999999 0 -0.0325 rpy=0 0 0
- joint Joint4: origin xyz=0.2542156431175849 0 0.0325 rpy=0 0 3.1416 -> xyz=0.47835000000000005 0 0.0325 rpy=0 0 3.1416

Commit message: add test point c

File: dynamics/src/dynamics/urdf/single_arm_v12.urdf (robot description, URDF)
Before this commit: robot single_arm_v12, 8 links, 7 joints
Links:
- link Link2: mass 0.5138042752232314 -> 0.478163838060215
- link Link3: mass 0.46633726625192845 -> 0.441060161173263
Joints:
- joint Joint3: origin xyz=0.5096499999999999 0 -0.0325 rpy=0 0 0 -> xyz=0.369235515941162 0 -0.0325 rpy=0 0 0
- joint Joint4: origin xyz=0.47835000000000005 0 0.0325 rpy=0 0 3.1416 -> xyz=0.378764484058838 0 0.0325 rpy=0 0 3.1416

File: dynamics/src/dynamics/urdf/single_arm_v12_motion.urdf (robot description, URDF)
Before this commit: robot single_arm_v12, 8 links, 7 joints
Links:
- link Link2: mass 0.5138042752232314 -> 0.478163838060215
- link Link3: mass 0.46633726625192845 -> 0.441060161173263
Joints:
- joint Joint3: origin xyz=0.5096499999999999 0 -0.0325 rpy=0 0 0 -> xyz=0.369235515941162 0 -0.0325 rpy=0 0 0
- joint Joint4: origin xyz=0.47835000000000005 0 0.0325 rpy=0 0 3.1416 -> xyz=0.378764484058838 0 0.0325 rpy=0 0 3.1416

Commit message: add original test case1

File: dynamics/src/dynamics/urdf/single_arm_v12.urdf (robot description, URDF)
Before this commit: robot single_arm_v12, 8 links, 7 joints
Links:
- link Link2: mass 0.478163838060215 -> 0.47438808875114563
- link Link3: mass 0.441060161173263 -> 0.42960652442301844
Joints:
- joint Joint3: origin xyz=0.369235515941162 0 -0.0325 rpy=0 0 0 -> xyz=0.35436 0 -0.0325 rpy=0 0 0
- joint Joint4: origin xyz=0.378764484058838 0 0.0325 rpy=0 0 3.1416 -> xyz=0.33364 0 0.0325 rpy=0 0 3.1416

File: dynamics/src/dynamics/urdf/single_arm_v12_motion.urdf (robot description, URDF)
Before this commit: robot single_arm_v12, 8 links, 7 joints
Links:
- link Link2: mass 0.478163838060215 -> 0.47438808875114563
- link Link3: mass 0.441060161173263 -> 0.42960652442301844
Joints:
- joint Joint3: origin xyz=0.369235515941162 0 -0.0325 rpy=0 0 0 -> xyz=0.35436 0 -0.0325 rpy=0 0 0
- joint Joint4: origin xyz=0.378764484058838 0 0.0325 rpy=0 0 3.1416 -> xyz=0.33364 0 0.0325 rpy=0 0 3.1416
