Commit message: add single_arm v19 test fix urdf fail

File: dynamics/src/dynamics/urdf/single_arm_v19_motion.urdf (robot description, URDF)
Before this commit: robot single_arm_v12, 8 links, 7 joints
Links:
- removed link Link1
- removed link Link2
- removed link Link3
- removed link Link4
- removed link Link5
- removed link Link6
- added link link1, mass 0.93428; collision mesh filename=package://single_arm_v19/meshes/link1.STL; visual mesh filename=package://single_arm_v19/meshes/link1.STL
- added link link2, mass 0.4749073641101881; collision mesh filename=package://single_arm_v19/meshes/link2.STL; visual mesh filename=package://dynamics/src/dynamics/meshes/merged_single_arm_v1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
- added link link3, mass 0.45080484472603943; collision mesh filename=package://single_arm_v19/meshes/link3.STL; visual mesh filename=package://dynamics/src/dynamics/meshes/merged_single_arm_v1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
- added link link4, mass 0.36924; collision mesh filename=package://single_arm_v19/meshes/link4.STL; visual mesh filename=package://single_arm_v19/meshes/link4.STL
- added link link5, mass 0.36821; collision mesh filename=package://single_arm_v19/meshes/link5.STL; visual mesh filename=package://single_arm_v19/meshes/link5.STL
- added link link6, mass 0.025977; collision mesh filename=package://single_arm_v19/meshes/link6.STL; visual mesh filename=package://single_arm_v19/meshes/link6.STL
- link base_link: mass 0.47711 -> 2.94316; geometry collision mesh filename=package://single_arm_v19/meshes/base_link.STL; visual mesh filename=package://single_arm_v19/meshes/base_link.STL
Joints:
- removed joint Joint1
- removed joint Joint2
- removed joint Joint3
- removed joint Joint4
- removed joint Joint5
- removed joint Joint6
- added joint joint1: type revolute, parent base_link, child link1, origin xyz=0 0 0.1445 rpy=0 0 0, axis 0 0 1, limit lower=-3.14 upper=3.14 effort=0 velocity=0
- added joint joint2: type revolute, parent link1, child link2, origin xyz=0 -0.0685 0.0315 rpy=1.5708 0 0, axis 0 0 1, limit lower=-3.14 upper=3.14 effort=0 velocity=0
- added joint joint3: type revolute, parent link2, child link3, origin xyz=0 0.346667000820369 -0.039 rpy=-3.1416 0 1.5708, axis 0 0 1, limit lower=-3.14 upper=3.14 effort=0 velocity=0
- added joint joint4: type revolute, parent link3, child link4, origin xyz=0.37323299917963104 0 -0.039 rpy=-3.1416 0 1.5708, axis 0 0 1, limit lower=-3.14 upper=3.14 effort=0 velocity=0
- added joint joint5: type revolute, parent link4, child link5, origin xyz=0 -0.052 0.0286 rpy=1.5708 1.5708 0, axis 0 0 1, limit lower=-3.14 upper=3.14 effort=0 velocity=0
- added joint joint6: type revolute, parent link5, child link6, origin xyz=-0.055 0 0.033001 rpy=3.1416 -1.5708 0, axis 0 0 -1, limit lower=-3.14 upper=3.14 effort=0 velocity=0

File: single_arm_v19/urdf/single_arm_v19.urdf (robot description, URDF)
Before this commit: robot single_arm_v12, 8 links, 7 joints
Links:
- removed link Link1
- removed link Link2
- removed link Link3
- removed link Link4
- removed link Link5
- removed link Link6
- added link link1, mass 0.93428; collision mesh filename=package://single_arm_v19/meshes/link1.STL; visual mesh filename=package://single_arm_v19/meshes/link1.STL
- added link link2, mass 0.4749073641101881; collision mesh filename=package://single_arm_v19/meshes/link2.STL; visual mesh filename=package://dynamics/src/dynamics/meshes/single_arm_v19_2_19.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
- added link link3, mass 0.45080484472603943; collision mesh filename=package://single_arm_v19/meshes/link3.STL; visual mesh filename=package://dynamics/src/dynamics/meshes/single_arm_v19_3_19.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
- added link link4, mass 0.36924; collision mesh filename=package://single_arm_v19/meshes/link4.STL; visual mesh filename=package://single_arm_v19/meshes/link4.STL
- added link link5, mass 0.36821; collision mesh filename=package://single_arm_v19/meshes/link5.STL; visual mesh filename=package://single_arm_v19/meshes/link5.STL
- added link link6, mass 0.025977; collision mesh filename=package://single_arm_v19/meshes/link6.STL; visual mesh filename=package://single_arm_v19/meshes/link6.STL
- link base_link: mass 0.47711 -> 2.94316; geometry collision mesh filename=package://single_arm_v19/meshes/base_link.STL; visual mesh filename=package://single_arm_v19/meshes/base_link.STL
Joints:
- removed joint Joint1
- removed joint Joint2
- removed joint Joint3
- removed joint Joint4
- removed joint Joint5
- removed joint Joint6
- added joint joint1: type revolute, parent base_link, child link1, origin xyz=0 0 0.1445 rpy=0 0 0, axis 0 0 1, limit lower=-3.14 upper=3.14 effort=0 velocity=0
- added joint joint2: type revolute, parent link1, child link2, origin xyz=0 -0.0685 0.0315 rpy=1.5708 0 0, axis 0 0 1, limit lower=-3.14 upper=3.14 effort=0 velocity=0
- added joint joint3: type revolute, parent link2, child link3, origin xyz=0 0.346667000820369 -0.039 rpy=-3.1416 0 1.5708, axis 0 0 1, limit lower=-3.14 upper=3.14 effort=0 velocity=0
- added joint joint4: type revolute, parent link3, child link4, origin xyz=0.37323299917963104 0 -0.039 rpy=-3.1416 0 1.5708, axis 0 0 1, limit lower=-3.14 upper=3.14 effort=0 velocity=0
- added joint joint5: type revolute, parent link4, child link5, origin xyz=0 -0.052 0.0286 rpy=1.5708 1.5708 0, axis 0 0 1, limit lower=-3.14 upper=3.14 effort=0 velocity=0
- added joint joint6: type revolute, parent link5, child link6, origin xyz=-0.055 0 0.033001 rpy=3.1416 -1.5708 0, axis 0 0 -1, limit lower=-3.14 upper=3.14 effort=0 velocity=0
