Commit message: fixed real robot to simulation urdf & not test

File: dynamics/src/dynamics/urdf/single_arm_v22_19cm_motion.urdf (robot description, URDF)
Before this commit: robot single_arm_v19, 7 links, 6 joints
Links:
- added link dummy
- link base_link: geometry collision mesh filename=package://single_arm_v22_19cm/meshes/base_link.STL; visual mesh filename=package://single_arm_v22_19cm/meshes/base_link.STL
- link link1: geometry collision mesh filename=package://single_arm_v22_19cm/meshes/link1.STL; visual mesh filename=package://single_arm_v22_19cm/meshes/link1.STL
- link link2: geometry collision mesh filename=package://dynamics/src/dynamics/meshes/merged_single_arm_v2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; visual mesh filename=package://dynamics/src/dynamics/meshes/merged_single_arm_v2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
- link link3: geometry collision mesh filename=package://dynamics/src/dynamics/meshes/merged_single_arm_v2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; visual mesh filename=package://dynamics/src/dynamics/meshes/merged_single_arm_v2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
- link link4: geometry collision mesh filename=package://single_arm_v22_19cm/meshes/link4.STL; visual mesh filename=package://single_arm_v22_19cm/meshes/link4.STL
- link link5: geometry collision mesh filename=package://single_arm_v22_19cm/meshes/link5.STL; visual mesh filename=package://single_arm_v22_19cm/meshes/link5.STL
- link link6: mass 0.025977 -> 0.0259770442543706; geometry collision mesh filename=package://single_arm_v22_19cm/meshes/link6.STL; visual mesh filename=package://single_arm_v22_19cm/meshes/link6.STL
Joints:
- added joint dummy_joint: type fixed, parent dummy, child base_link
- joint joint3: axis 0 0 1 -> 0 0 -1; origin xyz=0.2675 0 -0.039 rpy=-3.1416 0 1.5708 -> xyz=0.19 0 -0.0390000000000001 rpy=0 0 0
- joint joint4: origin xyz=0 0.2324 -0.039 rpy=-3.1416 0 1.5708 -> xyz=0.19 0 0.0390000000000083 rpy=0 0 -3.14159265358979
- joint joint5: axis 0 0 1 -> 1 0 0; origin xyz=0 -0.052 0.0286 rpy=1.5708 1.5708 0 -> xyz=0 0.052 0.0286 rpy=1.5707963267949 0 1.5707963267949
- joint joint6: axis 0 0 -1 -> 0 0 1; origin xyz=-0.055 0 0.033001 rpy=3.1416 -1.5708 0 -> xyz=0.0330005379381037 0.0549999394444907 0 rpy=1.57079632679488 -1.5707963267949 0
