Commit message: fixed stl & urdf real robot test ok

File: dynamics/src/dynamics/urdf/single_arm_v22_19cm.urdf (robot description, URDF)
Before this commit: robot single_arm_v22_19cm, 8 links, 7 joints
Links:
- link link2: mass 1.07602 -> 0.425863893965481; geometry collision mesh filename=package://single_arm_v22_19cm/meshes/link2.STL; visual mesh filename=package://dynamics/src/dynamics/meshes/single_arm_v22_19cm_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
- link link3: mass 1.00039 -> 0.40574020713355463; geometry collision mesh filename=package://single_arm_v22_19cm/meshes/link3.STL; visual mesh filename=package://dynamics/src/dynamics/meshes/single_arm_v22_19cm_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
Joints:
- joint joint3: origin xyz=0.19 0 -0.0390000000000001 rpy=0 0 0 -> xyz=0.2 0 -0.039 rpy=0 0 0
- joint joint4: origin xyz=0.19 0 0.0390000000000083 rpy=0 0 -3.14159265358979 -> xyz=0.2 0 0.039 rpy=0 0 -3.14159265358979

File: dynamics/src/dynamics/urdf/single_arm_v22_19cm_motion.urdf (robot description, URDF)
Before this commit: robot single_arm_v22_19cm, 8 links, 7 joints
Links:
- link link2: mass 1.07602 -> 0.425863893965481
- link link3: mass 1.00039 -> 0.40574020713355463
Joints:
- joint joint3: origin xyz=0.19 0 -0.0390000000000001 rpy=0 0 0 -> xyz=0.2 0 -0.039 rpy=0 0 0
- joint joint4: origin xyz=0.19 0 0.0390000000000083 rpy=0 0 -3.14159265358979 -> xyz=0.2 0 0.039 rpy=0 0 -3.14159265358979

File: single_arm_v22_19cm/urdf/single_arm_v22_19cm.urdf (robot description, URDF)
Before this commit: robot single_arm_v22_19cm, 7 links, 6 joints
Links:
- added link dummy
- link link2: mass 1.07602 -> 0.4749073641101887; geometry collision mesh filename=package://single_arm_v22_19cm/meshes/link2.STL; visual mesh filename=package://dynamics/src/dynamics/meshes/single_arm_v22_19cm_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
- link link3: mass 1.00039 -> 0.4508048439271571; geometry collision mesh filename=package://single_arm_v22_19cm/meshes/link3.STL; visual mesh filename=package://dynamics/src/dynamics/meshes/single_arm_v22_19cm_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
Joints:
- added joint dummy_joint: type fixed, parent dummy, child base_link
- joint joint3: origin xyz=0.19 0 -0.0390000000000001 rpy=0 0 0 -> xyz=0.304267000820369 0 -0.039 rpy=0 0 0
- joint joint4: origin xyz=0.19 0 0.0390000000000083 rpy=0 0 -3.14159265358979 -> xyz=0.29573299917963103 0 0.039 rpy=0 0 -3.14159265358979

Commit message: fixed stl read mass error

File: dynamics/src/dynamics/urdf/single_arm_v22_19cm.urdf (robot description, URDF)
Before this commit: robot single_arm_v22_19cm, 8 links, 7 joints
Links:
- link link2: mass 0.425863893965481 -> 1.33974234835036
- link link3: mass 0.40574020713355463 -> 1.19767908022107
Joints:
- joint joint3: origin xyz=0.2 0 -0.039 rpy=0 0 0 -> xyz=0.214867681425003 0 -0.039 rpy=0 0 0
- joint joint4: origin xyz=0.2 0 0.039 rpy=0 0 -3.14159265358979 -> xyz=0.285132318574997 0 0.039 rpy=0 0 -3.14159265358979

File: dynamics/src/dynamics/urdf/single_arm_v22_19cm_motion.urdf (robot description, URDF)
Before this commit: robot single_arm_v22_19cm, 8 links, 7 joints
Links:
- link link2: mass 0.425863893965481 -> 1.33974234835036
- link link3: mass 0.40574020713355463 -> 1.19767908022107
Joints:
- joint joint3: origin xyz=0.2 0 -0.039 rpy=0 0 0 -> xyz=0.214867681425003 0 -0.039 rpy=0 0 0
- joint joint4: origin xyz=0.2 0 0.039 rpy=0 0 -3.14159265358979 -> xyz=0.285132318574997 0 0.039 rpy=0 0 -3.14159265358979
